File: hw/kicad/laser_lipo.kicad_pcb (KiCad board)
At the start: 2 copper layers, 27.7 x 12.6 mm, 14 parts, among them J1 USB-MINI-B, P1 BAT+, P2 BAT-, P3 LZR+, P4 LZR-, SW1 SWITCH_INV, U1 MCP73831, U2 LP3985

Commit message: - finish pcb - add drill and gerbers, need to check them
Parts:
- moved P3 0.30 mm to (74.5, 46.9)
- moved R2 0.30 mm to (59.8, 47.3)
- moved P4 0.30 mm to (74.5, 56.7)
- turned D1 to 0 degrees
Routing:
- net GND: track 0.00 -> 56.7 mm, vias 0 -> 2
- net VBAT+: track 0.00 -> 20.6 mm, vias 0 -> 3
- net USB_VBUS: track 0.00 -> 8.72 mm, vias 0 -> 2
- net N-000008: track 0.00 -> 8.17 mm
- net N-0000011: track 0.00 -> 7.95 mm, vias 0 -> 2
- net N-000006: track 0.00 -> 5.71 mm
- net N-000007: track 0.00 -> 2.65 mm
- net N-0000010: track 0.00 -> 2.51 mm
- net N-0000013: track 0.00 -> 2.49 mm
- added copper zone on B.Cu, net GND
- added copper zone on F.Cu, net GND
Other:
- board size 27.7 x 12.6 mm -> 27.7 x 14.4 mm
- rule via_min_drill: 0.508 -> 0.3302
- rule via_min_size: 0.889 -> 0.6858
- board text added: "https://github.com/noahp/laser_lipo v0.0 2013-05"
