File: hw/kicad/laser_lipo.kicad_pcb (KiCad board)
At the start: 2 copper layers, 27.7 x 14.4 mm, 14 parts, among them J1 USB-MINI-B, P1 BAT+, P2 BAT-, P3 LZR+, P4 LZR-, SW1 SWITCH_INV, U1 MCP73831, U2 LP3985

Commit message: - add output archive - tidy up a bit
Routing:
- net GND: track 56.7 -> 10.3 mm, vias 2 -> 0
Changed lines of the file:
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@@
   (general
     (links 23)
-    (no_connects 0)
+    (no_connects 1)
     (area 50.170999 43.971 78.175001 60.629)
     (thickness 1.6)
     (drawings 11)
-    (tracks 75)
+    (tracks 52)
     (zones 0)
     (modules 14)
@@
   (gr_circle (center 58.6 53) (end 58.6 53.1) (layer F.SilkS) (width 0.2))
   (gr_circle (center 66.6 50.7) (end 66.6 50.8) (layer F.SilkS) (width 0.2))
-  (segment (start 68.25 50) (end 68.25 49.45) (width 0.254) (layer F.Cu) (net 1))
-  (segment (start 74.5 53.5) (end 74.5 56.7) (width 0.254) (layer F.Cu) (net 1) (status 20))
-  (segment (start 70 49) (end 74.5 53.5) (width 0.254) (layer F.Cu) (net 1))
-  (segment (start 68.7 49) (end 70 49) (width 0.254) (layer F.Cu) (net 1))
-  (segment (start 68.25 49.45) (end 68.7 49) (width 0.254) (layer F.Cu) (net 1))
   (segment (start 65.4 51.8) (end 67.4 51.8) (width 0.254) (layer F.Cu) (net 1))
+  (segment (start 65.4 51.8) (end 65.4 52.138) (width 0.254) (layer F.Cu) (net 1))
+  (segment (start 65.4 52.138) (end 64.538 53) (width 0.254) (layer F.Cu) (net 1))
+  (segment (start 67.4 51.8) (end 68.25 50.95) (width 0.254) (layer F.Cu) (net 1))
   (segment (start 68.25 50.95) (end 68.25 50) (width 0.254) (layer F.Cu) (net 1))
-  (segment (start 67.4 51.8) (end 68.25 50.95) (width 0.254) (layer F.Cu) (net 1))
-  (segment (start 63.2 46.538) (end 64.338 46.538) (width 0.254) (layer F.Cu) (net 1))
-  (segment (start 65.4 52.138) (end 64.538 53) (width 0.254) (layer F.Cu) (net 1))
-  (segment (start 65.4 47.6) (end 65.4 51.8) (width 0.254) (layer F.Cu) (net 1))
-  (segment (start 65.4 51.8) (end 65.4 52.138) (width 0.254) (layer F.Cu) (net 1))
-  (segment (start 64.338 46.538) (end 65.4 47.6) (width 0.254) (layer F.Cu) (net 1))
-  (segment (start 54.1 47.6) (end 54.1 56) (width 0.254) (layer F.Cu) (net 1))
-  (via (at 61.7 47.6) (size 0.6858) (drill 0.3302) (layers F.Cu B.Cu) (net 1))
-  (via (at 57.1 47.6) (size 0.6858) (drill 0.3302) (layers F.Cu B.Cu) (net 1))
-  (segment (start 61.7 47.6) (end 57.1 47.6) (width 0.254) (layer B.Cu) (net 1))
-  (segment (start 57.1 47.6) (end 54.1 47.6) (width 0.254) (layer F.Cu) (net 1))
-  (segment (start 61.7 47.6) (end 62.762 46.538) (width 0.254) (layer F.Cu) (net 1))
-  (segment (start 62.762 46.538) (end 63.2 46.538) (width 0.254) (layer F.Cu) (net 1))
-  (segment (start 61.4 47.3) (end 60.562 47.3) (width 0.254) (layer F.Cu) (net 1))
-  (segment (start 61.7 47.6) (end 61.4 47.3) (width 0.254) (layer F.Cu) (net 1))
-  (segment (start 59.938 54.9) (end 59.938 53.662) (width 0.254) (layer F.Cu) (net 1))
-  (segment (start 59.938 53.662) (end 60.25 53.35) (width 0.254) (layer F.Cu) (net 1))
-  (segment (start 59.938 54.9) (end 59.938 56.862) (width 0.254) (layer F.Cu) (net 1))
-  (segment (start 59.938 56.862) (end 59.2 57.6) (width 0.254) (layer F.Cu) (net 1))
-  (segment (start 60.25 53.35) (end 56.65 53.35) (width 0.254) (layer F.Cu) (net 1))
-  (segment (start 56.65 53.35) (end 56.6 53.4) (width 0.254) (layer F.Cu) (net 1))
-  (segment (start 60.25 52.4) (end 60.25 53.35) (width 0.254) (layer F.Cu) (net 1))
-  (segment (start 56.6 53.4) (end 56.6 53.5) (width 0.254) (layer F.Cu) (net 1))
-  (segment (start 56.6 53.5) (end 54.1 56) (width 0.254) (layer F.Cu) (net 1))
+  (segment (start 56.6 53.4) (end 60.2 53.4) (width 0.254) (layer F.Cu) (net 1))
+  (segment (start 60.25 53.35) (end 60.25 52.4) (width 0.254) (layer F.Cu) (net 1))
+  (segment (start 60.2 53.4) (end 60.25 53.35) (width 0.254) (layer F.Cu) (net 1))
   (segment (start 59.3 49.7) (end 59.038 49.438) (width 0.254) (layer F.Cu) (net 2))
   (segment (start 59.038 49.438) (end 59.038 47.3) (width 0.254) (layer F.Cu) (net 2))

Commit message: - v0.1 - add 1uF cap to output of 3.3v reg
Parts:
- added C3: 1uF, SM0603, F.Cu at (65.4, 47.4)
Routing:
- net N-000008: track 8.17 -> 10.4 mm
Other:
- board text added: "https://github.com/noahp/laser_lipo v0.1 2013-05"
- board text removed: "https://github.com/noahp/laser_lipo v0.0 2013-05"
Changed lines of the file:
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@@
-(kicad_pcb (version 3) (host pcbnew "(2013-03-31 BZR 4008)-stable")
+(kicad_pcb (version 3) (host pcbnew "(2013-03-04 BZR 3984)-stable")
   (general
-    (links 23)
+    (links 25)
     (no_connects 1)
-    (area 50.170999 43.971 78.175001 60.629)
+    (area 50.324999 44.524999 78.175001 59.075001)
     (thickness 1.6)
     (drawings 11)
-    (tracks 52)
+    (tracks 54)
     (zones 0)
-    (modules 14)
+    (modules 15)
     (nets 10)
   )
@@
   (net 2 N-0000010)
   (net 3 N-0000011)
-  (net 4 N-0000013)
-  (net 5 N-000006)
-  (net 6 N-000007)
-  (net 7 N-000008)
+  (net 4 N-0000012)
+  (net 5 N-000007)
+  (net 6 N-000008)
+  (net 7 N-000009)
   (net 8 USB_VBUS)
   (net 9 VBAT+)
@@
     (add_net N-0000010)
     (add_net N-0000011)
-    (add_net N-0000013)
-    (add_net N-000006)
+    (add_net N-0000012)
     (add_net N-000007)
     (add_net N-000008)
+    (add_net N-000009)
     (add_net USB_VBUS)
     (add_net VBAT+)
@@
     (pad 1 thru_hole circle (at 0 0) (size 1.75 1.75) (drill 1.02)
       (layers *.Cu *.Mask F.SilkS)
-      (net 7 N-000008)
+      (net 6 N-000008)
     )
   )
@@
     (pad 2 smd rect (at 0.75 -1.75) (size 0.7 1.5)
       (layers F.Cu F.Paste F.Mask)
-      (net 5 N-000006)
+      (net 7 N-000009)
     )
     (pad 3 smd rect (at 2.25 -1.75) (size 0.7 1.5)
@@
     (pad 1 smd rect (at -2.25 -1.75) (size 0.7 1.5)
       (layers F.Cu F.Paste F.Mask)
-      (net 6 N-000007)
+      (net 5 N-000007)
     )
   )
@@
     (pad 2 smd rect (at 0.762 0) (size 0.635 1.143)
       (layers F.Cu F.Paste F.Mask)
-      (net 4 N-0000013)
+      (net 3 N-0000011)
     )
     (model smd\resistors\R0603.wrl
@@
     (pad 1 smd rect (at -0.762 0 270) (size 0.635 1.143)
       (layers F.Cu F.Paste F.Mask)
-      (net 4 N-0000013)
+      (net 3 N-0000011)
     )
     (pad 2 smd rect (at 0.762 0 270) (size 0.635 1.143)
       (layers F.Cu F.Paste F.Mask)
-      (net 3 N-0000011)
+      (net 4 N-0000012)
     )
     (model smd\resistors\R0603.wrl
@@
     (pad 1 smd rect (at -0.762 0 180) (size 0.635 1.143)
       (layers F.Cu F.Paste F.Mask)
-      (net 6 N-000007)
+      (net 5 N-000007)
     )
     (pad 2 smd rect (at 0.762 0 180) (size 0.635 1.143)
@@
     (pad 1 smd rect (at 0 0) (size 0.55 1)
       (layers F.Cu F.Paste F.Mask)
-      (net 3 N-0000011)
+      (net 4 N-0000012)
     )
     (pad 2 smd rect (at 0.95 0) (size 0.55 1)
@@
     (pad 3 smd rect (at 1.9 0) (size 0.55 1)
       (layers F.Cu F.Paste F.Mask)
-      (net 5 N-000006)
+      (net 7 N-000009)
     )
     (pad 4 smd rect (at 1.9 -2.7) (size 0.55 1)
@@
     (pad 5 smd rect (at 0 -2.7) (size 0.55 1)
       (layers F.Cu F.Paste F.Mask)
-      (net 7 N-000008)
+      (net 6 N-000008)
     )
   )
@@
     )
   )
-  (gr_text "https://github.com/noahp/laser_lipo\nv0.0\n2013-05" (at 64.4 50.5) (layer B.SilkS)
+  (module SM0603 (layer F.Cu)
+    (at 65.405 47.371 90)
+    (attr smd)
+    (fp_text reference C3 (at 0 0 90) (layer F.SilkS)
+      (effects (font (size 0.508 0.4572) (thickness 0.1143)))
+    )
+    (fp_text value 1uF (at 0 0 90) (layer F.SilkS) hide
+      (effects (font (size 0.508 0.4572) (thickness 0.1143)))
+    )
+    (fp_line (start -1.143 -0.635) (end 1.143 -0.635) (layer F.SilkS) (width 0.127))
+    (fp_line (start 1.143 -0.635) (end 1.143 0.635) (layer F.SilkS) (width 0.127))
+    (fp_line (start 1.143 0.635) (end -1.143 0.635) (layer F.SilkS) (width 0.127))
+    (fp_line (start -1.143 0.635) (end -1.143 -0.635) (layer F.SilkS) (width 0.127))
+    (pad 1 smd rect (at -0.762 0 90) (size 0.635 1.143)
+      (layers F.Cu F.Paste F.Mask)
+      (net 6 N-000008)
+    )
+    (pad 2 smd rect (at 0.762 0 90) (size 0.635 1.143)
+      (layers F.Cu F.Paste F.Mask)
+      (net 1 GND)
+    )
+    (model smd\resistors\R0603.wrl
+      (at (xyz 0 0 0.001))
+      (scale (xyz 0.5 0.5 0.5))
+      (rotate (xyz 0 0 0))
+    )
+  )
+  (gr_text "https://github.com/noahp/laser_lipo\nv0.1\n2013-05" (at 64.4 50.5) (layer B.SilkS)
     (effects (font (size 0.8 0.8) (thickness 0.2)) (justify mirror))
   )
@@
   (segment (start 59.3 49.7) (end 59.038 49.438) (width 0.254) (layer F.Cu) (net 2))
   (segment (start 59.038 49.438) (end 59.038 47.3) (width 0.254) (layer F.Cu) (net 2))
-  (segment (start 59.3 52.4) (end 58.2 52.4) (width 0.254) (layer F.Cu) (net 3))
-  (segment (start 62.9 54.6) (end 62.9 53.362) (width 0.254) (layer F.Cu) (net 3))
-  (via (at 62.9 54.6) (size 0.6858) (drill 0.3302) (layers F.Cu B.Cu) (net 3))
-  (segment (start 60.7 52.4) (end 62.9 54.6) (width 0.254) (layer B.Cu) (net 3))
-  (segment (start 58.2 52.4) (end 60.7 52.4) (width 0.254) (layer B.Cu) (net 3))
-  (via (at 58.2 52.4) (size 0.6858) (drill 0.3302) (layers F.Cu B.Cu) (net 3))
-  (segment (start 64.462 50) (end 64.462 50.276) (width 0.254) (layer F.Cu) (net 4))
-  (segment (start 64.462 50.276) (end 62.9 51.838) (width 0.254) (layer F.Cu) (net 4))
-  (segment (start 69.2 50) (end 69.2 55.5) (width 0.254) (layer F.Cu) (net 5))
-  (segment (start 69.2 55.5) (end 69.05 55.65) (width 0.254) (layer F.Cu) (net 5))
-  (segment (start 66.062 53) (end 66.062 55.638) (width 0.254) (layer F.Cu) (net 6))
-  (segment (start 66.062 55.638) (end 66.05 55.65) (width 0.254) (layer F.Cu) (net 6))
-  (segment (start 67.3 47.3) (end 68.4 48.3) (width 0.254) (layer F.Cu) (net 7))
-  (segment (start 73.1 48.3) (end 74.5 46.9) (width 0.254) (layer F.Cu) (net 7) (status 20))
-  (segment (start 68.4 48.3) (end 73.1 48.3) (width 0.254) (layer F.Cu) (net 7))
+  (segment (start 64.462 50) (end 64.462 50.276) (width 0.254) (layer F.Cu) (net 3))
+  (segment (start 64.462 50.276) (end 62.9 51.838) (width 0.254) (layer F.Cu) (net 3))
+  (segment (start 59.3 52.4) (end 58.2 52.4) (width 0.254) (layer F.Cu) (net 4))
+  (segment (start 62.9 54.6) (end 62.9 53.362) (width 0.254) (layer F.Cu) (net 4))
+  (via (at 62.9 54.6) (size 0.6858) (drill 0.3302) (layers F.Cu B.Cu) (net 4))
+  (segment (start 60.7 52.4) (end 62.9 54.6) (width 0.254) (layer B.Cu) (net 4))
+  (segment (start 58.2 52.4) (end 60.7 52.4) (width 0.254) (layer B.Cu) (net 4))
+  (via (at 58.2 52.4) (size 0.6858) (drill 0.3302) (layers F.Cu B.Cu) (net 4))
+  (segment (start 66.062 53) (end 66.062 55.638) (width 0.254) (layer F.Cu) (net 5))
+  (segment (start 66.062 55.638) (end 66.05 55.65) (width 0.254) (layer F.Cu) (net 5))
+  (segment (start 67.3 47.3) (end 66.467 48.133) (width 0.254) (layer F.Cu) (net 6))
+  (segment (start 66.467 48.133) (end 65.405 48.133) (width 0.254) (layer F.Cu) (net 6))
+  (segment (start 67.3 47.3) (end 68.4 48.3) (width 0.254) (layer F.Cu) (net 6))
+  (segment (start 73.1 48.3) (end 74.5 46.9) (width 0.254) (layer F.Cu) (net 6) (status 20))
+  (segment (start 68.4 48.3) (end 73.1 48.3) (width 0.254) (layer F.Cu) (net 6))
+  (segment (start 69.2 50) (end 69.2 55.5) (width 0.254) (layer F.Cu) (net 7))
+  (segment (start 69.2 55.5) (end 69.05 55.65) (width 0.254) (layer F.Cu) (net 7))
   (segment (start 63.2 48.062) (end 62.938 48.324) (width 0.254) (layer F.Cu) (net 8))
   (segment (start 62.938 48.324) (end 62.938 50) (width 0.254) (layer F.Cu) (net 8))

Commit message: - need to connect 3.3v regulator to gnd >_<
Routing:
- net GND: track 10.3 -> 12.2 mm, vias 0 -> 1
Changed lines of the file:
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@@
   (general
     (links 25)
-    (no_connects 1)
-    (area 50.324999 44.524999 78.175001 59.075001)
+    (no_connects 0)
+    (area 50.170999 43.971 78.175001 60.629)
     (thickness 1.6)
     (drawings 11)
-    (tracks 54)
+    (tracks 57)
     (zones 0)
     (modules 15)
@@
   (gr_circle (center 58.6 53) (end 58.6 53.1) (layer F.SilkS) (width 0.2))
   (gr_circle (center 66.6 50.7) (end 66.6 50.8) (layer F.SilkS) (width 0.2))
+  (segment (start 64.538 53) (end 64.538 54.842) (width 0.254) (layer F.Cu) (net 1))
+  (via (at 64.516 54.864) (size 0.6858) (drill 0.3302) (layers F.Cu B.Cu) (net 1))
+  (segment (start 64.538 54.842) (end 64.516 54.864) (width 0.254) (layer F.Cu) (net 1))
   (segment (start 65.4 51.8) (end 67.4 51.8) (width 0.254) (layer F.Cu) (net 1))
   (segment (start 65.4 51.8) (end 65.4 52.138) (width 0.254) (layer F.Cu) (net 1))
