File: hw/kicad/laser_lipo.sch (KiCad schematic (older format))
At the start: 14 parts, among them J1 USB-MINI-B, P1 BAT+, P2 BAT-, P3 LZR+, P4 LZR-, SW1 SW_PUSH, U1 MCP73831, U2 LP3985

Commit message: - add footprint for slide switch
Parts:
- removed SW1: SW_PUSH, ~, symbol SW_PUSH
- added SW?: SWITCH_INV, ~, symbol SWITCH_INV
Connections:
- wire segments 26 -> 28
Other:
- moved on the sheet: P3, P4, R3, U2
Changed lines of the file:
@@
-EESchema Schematic File Version 2  date 5/14/2013 8:00:28 AM
+EESchema Schematic File Version 2  date 5/14/2013 8:31:32 AM
 LIBS:power
 LIBS:device
@@
 LIBS:valves
 LIBS:kicadlib
+LIBS:laser_lipo-cache
 EELAYER 27 0
 EELAYER END
@@
 L LP3985 U2
 U 1 1 51922445
-P 6550 4800
-F 0 "U2" H 6550 4500 60  0000 C CNN
-F 1 "LP3985" H 6600 5100 60  0000 C CNN
-F 2 "~" H 6550 4800 60  0000 C CNN
-F 3 "~" H 6550 4800 60  0000 C CNN
-	1    6550 4800
+P 7200 4900
+F 0 "U2" H 7200 4600 60  0000 C CNN
+F 1 "LP3985" H 7250 5200 60  0000 C CNN
+F 2 "~" H 7200 4900 60  0000 C CNN
+F 3 "~" H 7200 4900 60  0000 C CNN
+	1    7200 4900
 	1    0    0    -1
 $EndComp
@@
 	1    0    0    -1
 $EndComp
-Wire Wire Line
-	4500 4950 5150 4950
 Wire Wire Line
 	5000 5600 5000 5350
@@
 L TST P3
 U 1 1 51922676
-P 7300 4550
-F 0 "P3" H 7300 4850 40  0000 C CNN
-F 1 "LZR+" H 7300 4800 30  0000 C CNN
-F 2 "~" H 7300 4550 60  0000 C CNN
-F 3 "~" H 7300 4550 60  0000 C CNN
-	1    7300 4550
+P 7950 4650
+F 0 "P3" H 7950 4950 40  0000 C CNN
+F 1 "LZR+" H 7950 4900 30  0000 C CNN
+F 2 "~" H 7950 4650 60  0000 C CNN
+F 3 "~" H 7950 4650 60  0000 C CNN
+	1    7950 4650
 	1    0    0    -1
 $EndComp
@@
 L TST P4
 U 1 1 51922683
-P 7450 4550
-F 0 "P4" H 7450 4850 40  0000 C CNN
-F 1 "LZR-" H 7450 4800 30  0000 C CNN
-F 2 "~" H 7450 4550 60  0000 C CNN
-F 3 "~" H 7450 4550 60  0000 C CNN
-	1    7450 4550
-	1    0    0    -1
-$EndComp
-$Comp
-L SW_PUSH SW1
-U 1 1 519226A4
-P 5450 4950
-F 0 "SW1" H 5600 5060 50  0000 C CNN
-F 1 "SW_PUSH" H 5450 4870 50  0000 C CNN
-F 2 "~" H 5450 4950 60  0000 C CNN
-F 3 "~" H 5450 4950 60  0000 C CNN
-	1    5450 4950
+P 8100 4650
+F 0 "P4" H 8100 4950 40  0000 C CNN
+F 1 "LZR-" H 8100 4900 30  0000 C CNN
+F 2 "~" H 8100 4650 60  0000 C CNN
+F 3 "~" H 8100 4650 60  0000 C CNN
+	1    8100 4650
 	1    0    0    -1
 $EndComp
 Connection ~ 5000 4950
-Wire Wire Line
-	5750 4950 5950 4950
 $Comp
 L R R3
 U 1 1 519226FA
-P 5850 5300
-F 0 "R3" V 5930 5300 40  0000 C CNN
-F 1 "2k" V 5857 5301 40  0000 C CNN
-F 2 "~" V 5780 5300 30  0000 C CNN
-F 3 "~" H 5850 5300 30  0000 C CNN
-	1    5850 5300
-	1    0    0    -1
-$EndComp
-Wire Wire Line
-	5850 4950 5850 5050
-Connection ~ 5850 4950
+P 5300 5500
+F 0 "R3" V 5380 5500 40  0000 C CNN
+F 1 "2k" V 5307 5501 40  0000 C CNN
+F 2 "~" V 5230 5500 30  0000 C CNN
+F 3 "~" H 5300 5500 30  0000 C CNN
+	1    5300 5500
+	1    0    0    -1
+$EndComp
 $Comp
 L GND #PWR04
 U 1 1 51922723
-P 5850 5650
-F 0 "#PWR04" H 5850 5650 30  0001 C CNN
-F 1 "GND" H 5850 5580 30  0001 C CNN
-F 2 "" H 5850 5650 60  0000 C CNN
-F 3 "" H 5850 5650 60  0000 C CNN
-	1    5850 5650
-	1    0    0    -1
-$EndComp
-Wire Wire Line
-	5850 5550 5850 5650
+P 5300 5850
+F 0 "#PWR04" H 5300 5850 30  0001 C CNN
+F 1 "GND" H 5300 5780 30  0001 C CNN
+F 2 "" H 5300 5850 60  0000 C CNN
+F 3 "" H 5300 5850 60  0000 C CNN
+	1    5300 5850
+	1    0    0    -1
+$EndComp
+Wire Wire Line
+	5300 5750 5300 5850
 $Comp
 L GND #PWR05
 U 1 1 51922742
-P 5850 4800
-F 0 "#PWR05" H 5850 4800 30  0001 C CNN
-F 1 "GND" H 5850 4730 30  0001 C CNN
-F 2 "" H 5850 4800 60  0000 C CNN
-F 3 "" H 5850 4800 60  0000 C CNN
-	1    5850 4800
-	1    0    0    -1
-$EndComp
-Wire Wire Line
-	5850 4800 5950 4800
-Wire Wire Line
-	4900 4650 5950 4650
+P 6500 4900
+F 0 "#PWR05" H 6500 4900 30  0001 C CNN
+F 1 "GND" H 6500 4830 30  0001 C CNN
+F 2 "" H 6500 4900 60  0000 C CNN
+F 3 "" H 6500 4900 60  0000 C CNN
+	1    6500 4900
+	1    0    0    -1
+$EndComp
+Wire Wire Line
+	6500 4900 6600 4900
 Wire Wire Line
 	5000 4650 5000 4950
 Text GLabel 4900 4650 0    60   Input ~ 0
 VBAT+
-Connection ~ 5000 4650
 $Comp
 L TST P2
@@
 Wire Wire Line
 	5150 3900 5250 3900
-NoConn ~ 7200 4950
+NoConn ~ 7850 5050
 $Comp
 L GND #PWR06
@@
 	5400 4050 5400 4150
 Wire Wire Line
-	7300 4550 7300 4650
-Wire Wire Line
-	7300 4650 7200 4650
+	7950 4650 7950 4750
+Wire Wire Line
+	7950 4750 7850 4750
 $Comp
 L GND #PWR07
 U 1 1 51922A06
-P 7450 4650
-F 0 "#PWR07" H 7450 4650 30  0001 C CNN
-F 1 "GND" H 7450 4580 30  0001 C CNN
-F 2 "" H 7450 4650 60  0000 C CNN
-F 3 "" H 7450 4650 60  0000 C CNN
-	1    7450 4650
-	1    0    0    -1
-$EndComp
-Wire Wire Line
-	7450 4550 7450 4650
+P 8100 4750
+F 0 "#PWR07" H 8100 4750 30  0001 C CNN
+F 1 "GND" H 8100 4680 30  0001 C CNN
+F 2 "" H 8100 4750 60  0000 C CNN
+F 3 "" H 8100 4750 60  0000 C CNN
+	1    8100 4750
+	1    0    0    -1
+$EndComp
+Wire Wire Line
+	8100 4650 8100 4750
+$Comp
+L SWITCH_INV SW?
+U 1 1 51922CEC
+P 5900 5050
+F 0 "SW?" H 5700 5200 50  0000 C CNN
+F 1 "SWITCH_INV" H 5750 4900 50  0000 C CNN
+F 2 "~" H 5900 5050 60  0000 C CNN
+F 3 "~" H 5900 5050 60  0000 C CNN
+	1    5900 5050
+	-1   0    0    1
+$EndComp
+Wire Wire Line
+	4500 4950 5400 4950
+Wire Wire Line
+	5300 5250 5300 5150
+Wire Wire Line
+	5300 5150 5400 5150
+Wire Wire Line
+	6600 5050 6400 5050
+Wire Wire Line
+	5000 4650 4900 4650
+Wire Wire Line
+	6600 4750 5000 4750
+Connection ~ 5000 4750
 $EndSCHEMATC

Commit message: - put footprints on pcb
Parts:
- gave numbers to parts that had none: 1
Changed lines of the file:
@@
-EESchema Schematic File Version 2  date 5/14/2013 8:31:32 AM
+EESchema Schematic File Version 2  date 5/14/2013 9:19:32 AM
 LIBS:power
 LIBS:device
@@
 	8100 4650 8100 4750
 $Comp
-L SWITCH_INV SW?
+L SWITCH_INV SW1
 U 1 1 51922CEC
 P 5900 5050
-F 0 "SW?" H 5700 5200 50  0000 C CNN
+F 0 "SW1" H 5700 5200 50  0000 C CNN
 F 1 "SWITCH_INV" H 5750 4900 50  0000 C CNN
 F 2 "~" H 5900 5050 60  0000 C CNN

Commit message: - v0.1 - add 1uF cap to output of 3.3v reg
Parts:
- added C3: 1uF, ~, symbol C
Connections:
- wire segments 28 -> 29
Other:
- moved on the sheet: P3, P4
Changed lines of the file:
@@
-EESchema Schematic File Version 2  date 5/14/2013 9:19:32 AM
+EESchema Schematic File Version 2  date 5/29/2013 11:34:53 AM
 LIBS:power
 LIBS:device
@@
 Sheet 1 1
 Title ""
-Date "14 may 2013"
+Date "29 may 2013"
 Rev ""
 Comp ""
@@
 L TST P3
 U 1 1 51922676
-P 7950 4650
-F 0 "P3" H 7950 4950 40  0000 C CNN
-F 1 "LZR+" H 7950 4900 30  0000 C CNN
-F 2 "~" H 7950 4650 60  0000 C CNN
-F 3 "~" H 7950 4650 60  0000 C CNN
-	1    7950 4650
+P 8200 4650
+F 0 "P3" H 8200 4950 40  0000 C CNN
+F 1 "LZR+" H 8200 4900 30  0000 C CNN
+F 2 "~" H 8200 4650 60  0000 C CNN
+F 3 "~" H 8200 4650 60  0000 C CNN
+	1    8200 4650
 	1    0    0    -1
 $EndComp
@@
 L TST P4
 U 1 1 51922683
-P 8100 4650
-F 0 "P4" H 8100 4950 40  0000 C CNN
-F 1 "LZR-" H 8100 4900 30  0000 C CNN
-F 2 "~" H 8100 4650 60  0000 C CNN
-F 3 "~" H 8100 4650 60  0000 C CNN
-	1    8100 4650
+P 8350 4650
+F 0 "P4" H 8350 4950 40  0000 C CNN
+F 1 "LZR-" H 8350 4900 30  0000 C CNN
+F 2 "~" H 8350 4650 60  0000 C CNN
+F 3 "~" H 8350 4650 60  0000 C CNN
+	1    8350 4650
 	1    0    0    -1
 $EndComp
@@
 Wire Wire Line
 	5400 4050 5400 4150
-Wire Wire Line
-	7950 4650 7950 4750
-Wire Wire Line
-	7950 4750 7850 4750
 $Comp
 L GND #PWR07
 U 1 1 51922A06
-P 8100 4750
-F 0 "#PWR07" H 8100 4750 30  0001 C CNN
-F 1 "GND" H 8100 4680 30  0001 C CNN
-F 2 "" H 8100 4750 60  0000 C CNN
-F 3 "" H 8100 4750 60  0000 C CNN
-	1    8100 4750
-	1    0    0    -1
-$EndComp
-Wire Wire Line
-	8100 4650 8100 4750
+P 8350 5250
+F 0 "#PWR07" H 8350 5250 30  0001 C CNN
+F 1 "GND" H 8350 5180 30  0001 C CNN
+F 2 "" H 8350 5250 60  0000 C CNN
+F 3 "" H 8350 5250 60  0000 C CNN
+	1    8350 5250
+	1    0    0    -1
+$EndComp
+Wire Wire Line
+	8350 4650 8350 5250
 $Comp
 L SWITCH_INV SW1
@@
 	6600 4750 5000 4750
 Connection ~ 5000 4750
+$Comp
+L C C3
+U 1 1 51A62082
+P 8100 4950
+F 0 "C3" H 8100 5050 40  0000 L CNN
+F 1 "1uF" H 8106 4865 40  0000 L CNN
+F 2 "~" H 8138 4800 30  0000 C CNN
+F 3 "~" H 8100 4950 60  0000 C CNN
+	1    8100 4950
+	1    0    0    -1
+$EndComp
+Wire Wire Line
+	7850 4750 8200 4750
+Wire Wire Line
+	8200 4750 8200 4650
+Connection ~ 8100 4750
+Wire Wire Line
+	8100 5150 8350 5150
+Connection ~ 8350 5150
 $EndSCHEMATC
